File: pcb/kicad/ergobox.kicad_pcb (KiCad board)
At the start: 2 copper layers, 234.6 x 150.2 mm, 80 parts, among them SW1 SW_Push, SW10 Kailh, SW11 Kailh, SW12 Kailh, SW13 Kailh, SW14 Kailh, SW15 Kailh, SW16 Kailh, SW17 Kailh, SW18 Kailh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

Commit message: fix: adjusts copper fills
Parts:
- moved D12 1.30 mm to (125.4, 152.2)
- moved D11 1.30 mm to (140.7, 119.7)
- moved D4 1.30 mm to (139.5, 80.7)
- moved D8 1.30 mm to (240.5, 84.2)
- moved D9 1.30 mm to (205.3, 91.6)
- moved SW17 1.30 mm to (140.7, 115.0)
- moved H5 1.30 mm to (143.2, 26.8)
- moved C6 1.30 mm to (65.8, 35.9)
- moved C16 1.30 mm to (54.5, 22.8)
- moved H1 1.30 mm to (32.5, 26.5)
- moved U2 1.30 mm to (60.5, 34.9)
- moved USB1 1.30 mm to (61.5, 14.5)
- moved C14 1.30 mm to (68.5, 23.3)
- moved C15 1.30 mm to (68.5, 28.5)
- moved D1 1.30 mm to (41.9, 63.0)
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Routing:
- net +1V1: track 27.1 -> 16.3 mm
- net +3V3: track 69.3 -> 65.7 mm, vias 2 -> 0
- net GND: track 20.4 -> 17.5 mm, vias 8 -> 10
- net +5V: track 16.9 -> 19.8 mm
- added copper zone on F.Cu, net +1V1
- added copper zone on F.Cu, net +5V

Commit message: feat: initial completed PCB layout
Parts:
- moved C23 224.1 mm to (237.5, 49.0), turned to 90 degrees
- moved C24 221.0 mm to (236.2, 88.0)
- moved H7 204.1 mm to (124.8, 95.9)
- moved C25 197.2 mm to (213.8, 90.0)
- moved C22 184.1 mm to (205.6, 56.8), turned to 180 degrees
- moved C28 174.3 mm to (133.7, 147.3), turned to 90 degrees
- moved C26 171.9 mm to (180.7, 98.6)
- moved C27 159.3 mm to (148.7, 114.6), turned to 90 degrees
- moved C21 155.4 mm to (169.8, 64.1), turned to 180 degrees
- moved C20 149.8 mm to (141.6, 85.0)
- moved C19 119.3 mm to (110.8, 89.4)
- moved C13 113.5 mm to (124.5, 44.9), turned to 90 degrees
- moved R5 108.7 mm to (124.5, 41.1), turned to 90 degrees
- moved C12 104.0 mm to (121.2, 41.0)
- moved R6 93.9 mm to (110.2, 31.4), turned to 90 degrees
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Routing:
- net +5V: track 19.8 -> 572.2 mm, vias 0 -> 2
- net BTN_K4: track 0.00 -> 129.5 mm, vias 0 -> 3
- net BTN_UP: track 0.00 -> 109.9 mm, vias 0 -> 1
- net BTN_P4: track 0.00 -> 107.9 mm, vias 0 -> 1
- net LED: track 0.00 -> 106.5 mm
- net BTN_K3: track 0.00 -> 99.5 mm, vias 0 -> 3
- net OPT6: track 0.00 -> 92.2 mm
- net BTN_LEFT: track 0.00 -> 91.8 mm, vias 0 -> 1
- net OPT5: track 0.00 -> 82.1 mm
- net BTN_P3: track 0.00 -> 77.1 mm, vias 0 -> 1
- net BTN_K1: track 0.00 -> 76.0 mm, vias 0 -> 3
- net BTN_K2: track 0.00 -> 74.2 mm, vias 0 -> 3
- net OPT4: track 0.00 -> 72.0 mm
- net GND: track 17.5 -> 81.3 mm, vias 10 -> 46
- net OPT3: track 0.00 -> 59.3 mm
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Other:
- outline, holes or cut-outs redrawn

Commit message: chore: adjusts aesthetics
Other:
- board text added: "BOOT"
- board text added: "ERGOBOX"
- board text added: "Hitbox-style fightstick"
- board text added: "RESET"
- board text added: "based from Flatbox 4"
- board text added: "derivative work from github.com/jfedor2/flatbox"
- board text added: "github.com/richardneililagan/ergobox"
- board text added: "ver 0.1.0.20220926"
Changed lines of the file:
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@@
     (property "Sheetname" "")
     (attr exclude_from_pos_files)
-    (fp_text reference "H2" (at 0 5.7) (layer "F.SilkS")
+    (fp_text reference "H2" (at 0 5.7) (layer "F.SilkS") hide
       (effects (font (size 1 1) (thickness 0.15)))
     )
@@
     (property "Sheetname" "")
     (attr exclude_from_pos_files)
-    (fp_text reference "H7" (at 0 -5.3) (layer "F.SilkS")
+    (fp_text reference "H7" (at 0 -5.3) (layer "F.SilkS") hide
       (effects (font (size 1 1) (thickness 0.15)))
     )
@@
     (property "Sheetname" "")
     (attr exclude_from_pos_files)
-    (fp_text reference "H3" (at 0 -5.3) (layer "F.SilkS")
+    (fp_text reference "H3" (at 0 -5.3) (layer "F.SilkS") hide
       (effects (font (size 1 1) (thickness 0.15)))
     )
@@
     (property "Sheetname" "")
     (attr exclude_from_pos_files)
-    (fp_text reference "H6" (at 0.2 -5.45) (layer "F.SilkS")
+    (fp_text reference "H6" (at 0.2 -5.45) (layer "F.SilkS") hide
       (effects (font (size 1 1) (thickness 0.15)))
     )
@@
     (property "Sheetname" "")
     (attr exclude_from_pos_files)
-    (fp_text reference "H4" (at 0 -5.3) (layer "F.SilkS")
+    (fp_text reference "H4" (at 0 -5.3) (layer "F.SilkS") hide
       (effects (font (size 1 1) (thickness 0.15)))
     )
@@
     (property "Sheetname" "")
     (attr exclude_from_pos_files)
-    (fp_text reference "H5" (at 0 5.8) (layer "F.SilkS")
+    (fp_text reference "H5" (at 0 5.8) (layer "F.SilkS") hide
       (effects (font (size 1 1) (thickness 0.15)))
     )
@@
     (property "Sheetname" "")
     (attr exclude_from_pos_files)
-    (fp_text reference "H1" (at 0 5.5) (layer "F.SilkS")
+    (fp_text reference "H1" (at 0 5.5) (layer "F.SilkS") hide
       (effects (font (size 1 1) (thickness 0.15)))
     )
@@
   (gr_circle (center -50.471077 83.823754) (end -39.058399 80.11555) (layer "F.SilkS") (width 0.15) (fill none))
   (gr_circle (center 424.3 102.2) (end 438.3 102.2) (layer "F.SilkS") (width 0.15) (fill none))
+  (gr_rect (start 242.4 123.1) (end 248.4 129.1) (layer "F.SilkS") (width 0.4) (fill none))
   (gr_circle (center 352.300001 102.2) (end 366.300001 102.2) (layer "F.SilkS") (width 0.15) (fill none))
   (gr_circle (center 205.254263 86.938806) (end 218.948329 84.028042) (layer "F.SilkS") (width 0.15) (fill none))
@@
   (gr_circle (center -101.890722 79.089839) (end -90.478042 75.381636) (layer "F.SilkS") (width 0.15) (fill none))
   (gr_circle (center 125.354263 147.538806) (end 141.354263 147.538806) (layer "F.SilkS") (width 0.15) (fill none))
+  (gr_poly
+    (pts
+      (xy 250.5 127)
+      (xy 248.4 127)
+      (xy 248.4 123.1)
+      (xy 244.9 123)
+      (xy 244.9 121)
+      (xy 250.5 121)
+    ) (layer "F.SilkS") (width 0.15) (fill solid))
   (gr_circle (center 326.3 77.8) (end 340.3 77.8) (layer "F.SilkS") (width 0.15) (fill none))
   (gr_circle (center 239.310011 40.339921) (end 253.004077 37.429157) (layer "F.SilkS") (width 0.15) (fill none))
@@
   (gr_line (start 32.454263 165.588806) (end 253.854263 165.538998) (layer "Edge.Cuts") (width 0.1))
   (gr_line (start 120.954263 15.438806) (end 131.954263 15.438806) (layer "Edge.Cuts") (width 0.1))
+  (gr_text "ver 0.1.0.20220926" (at 253.7 137.8 90) (layer "B.SilkS")
+    (effects (font (size 1.5 1.5) (thickness 0.15)) (justify mirror))
+  )
   (gr_text "UP" (at 125.354263 160.238806) (layer "F.SilkS")
     (effects (font (size 1 1) (thickness 0.15)))
@@
     (effects (font (size 1 1) (thickness 0.15)))
   )
+  (gr_text "Hitbox-style fightstick" (at 214.4 136.8) (layer "F.SilkS")
+    (effects (font (size 3 3) (thickness 0.5)))
+  )
+  (gr_text "ERGOBOX" (at 240.9 128.1) (layer "F.SilkS")
+    (effects (font (size 8 9) (thickness 1.3)) (justify right))
+  )
   (gr_text "P2" (at -74.042434 72.475086 18) (layer "F.SilkS")
     (effects (font (size 1 1) (thickness 0.15)))
@@
     (effects (font (size 1 1) (thickness 0.15)))
   )
+  (gr_text "derivative work from\ngithub.com/jfedor2/flatbox" (at 239.8 157.8) (layer "F.SilkS")
+    (effects (font (size 1.5 1.5) (thickness 0.15) italic) (justify right))
+  )
   (gr_text "K4" (at -18.219926 93.182347 18) (layer "F.SilkS")
     (effects (font (size 1 1) (thickness 0.15)))
@@
     (effects (font (size 1 1) (thickness 0.15)))
   )
+  (gr_text "based from Flatbox 4" (at 219.1 141.3) (layer "F.SilkS")
+    (effects (font (size 2.5 2.5) (thickness 0.3)))
+  )
   (gr_text "K4" (at 427.544678 112.186092 18) (layer "F.SilkS")
     (effects (font (size 1 1) (thickness 0.15)))
@@
     (effects (font (size 1 1) (thickness 0.15)))
   )
+  (gr_text "RESET" (at 115 49.5 90) (layer "F.SilkS")
+    (effects (font (size 1.5 1.5) (thickness 0.15)))
+  )
   (gr_text "K1" (at -99.410645 119.372187 18) (layer "F.SilkS")
     (effects (font (size 1 1) (thickness 0.15)))
@@
     (effects (font (size 1 1) (thickness 0.15)))
   )
+  (gr_text "github.com/richardneililagan/ergobox" (at 210.3 152.1) (layer "F.SilkS")
+    (effects (font (size 2 2) (thickness 0.15)))
+  )
+  (gr_text "BOOT" (at 115 42.6 90) (layer "F.SilkS")
+    (effects (font (size 1.5 1.5) (thickness 0.15)))
+  )
   (gr_text "P4" (at 434.544679 73.686093 18) (layer "F.SilkS")
